File: HP6632B_binding_posts.kicad_pcb (KiCad board)
At the start: 2 copper layers, 45 x 73 mm, 20 parts, among them J1 Conn_01x01, J615 Conn_01x04_Male

Commit message: better doc
Parts:
- C603, C604: value 4.7n -> 4.7n 250V
- C605, C606, C607, C608: value 220p -> 220p 1kV
