File: HP6632B_binding_posts.kicad_sch (KiCad schematic)
At the start: 20 parts, among them J1 Conn_01x01, J615 Conn_01x04_Male

Commit message: better doc
Parts:
- C603, C604: value 4.7n -> 4.7n 250V
- C605, C606, C607, C608: value 220p -> 220p 1kV
Changed lines of the file:
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@@
       (effects (font (size 1.27 1.27)) (justify left))
     )
-    (property "Value" "4.7n" (at 133.35 61.595 0)
+    (property "Value" "4.7n 250V" (at 133.35 61.595 0)
       (effects (font (size 1.27 1.27)) (justify left))
     )
@@
       (effects (font (size 1.27 1.27)) (justify left))
     )
-    (property "Value" "4.7n" (at 133.35 84.455 0)
+    (property "Value" "4.7n 250V" (at 133.35 84.455 0)
       (effects (font (size 1.27 1.27)) (justify left))
     )
@@
       (effects (font (size 1.27 1.27)) (justify left))
     )
-    (property "Value" "220p" (at 151.13 61.595 0)
+    (property "Value" "220p 1kV" (at 151.13 61.595 0)
       (effects (font (size 1.27 1.27)) (justify left))
     )
@@
       (effects (font (size 1.27 1.27)) (justify left))
     )
-    (property "Value" "220p" (at 151.13 84.455 0)
+    (property "Value" "220p 1kV" (at 151.13 84.455 0)
       (effects (font (size 1.27 1.27)) (justify left))
     )
@@
       (effects (font (size 1.27 1.27)) (justify left))
     )
-    (property "Value" "220p" (at 167.64 73.025 0)
+    (property "Value" "220p 1kV" (at 167.64 73.025 0)
       (effects (font (size 1.27 1.27)) (justify left))
     )
@@
       (effects (font (size 1.27 1.27)) (justify left))
     )
-    (property "Value" "220p" (at 167.64 95.885 0)
-      (effects (font (size 1.27 1.27)) (justify left))
-    )
+    (property "Value" "220p 1kV" (at 167.64 95.885 0)
+      (effects (font (size 1.27 1.27)) (justify left))
+    )
